Commit message: Move the origin to an orchard in Greece, add the datum script, add top-down tif + geotagged tif images, add the base station model near the origin

File: cpr_orchard_gazebo/urdf/orchard_geometry.urdf.xacro (robot description, xacro)
@@ -47,3 +47,7 @@
   </link>
   <gazebo> <static>true</static></gazebo>
+  <xacro:include filename="$(find cpr_accessories_gazebo)/urdf/base_station.urdf.xacro" />
+  <xacro:cpr_base_station name="base_station" parent="orchard_world_link">
+    <origin xyz="1 2 0" />
+  </xacro:cpr_base_station>
 </robot>
