Commit message: Add the water mesh to the visualization since UUV is disabled. This way the water at least renders, even if it doesn't have any physics

File: cpr_inspection_gazebo/urdf/inspection_geometry.urdf.xacro (robot description, xacro)
@@ -11,4 +11,10 @@
       <geometry>
         <mesh filename="package://cpr_inspection_gazebo/meshes/inspection_world.dae"/>
+      </geometry>
+    </visual>
+    <visual>
+      <origin xyz="0 0 0" rpy="0 0 0"/>
+      <geometry>
+        <mesh filename="package://cpr_inspection_gazebo/meshes/inspection_water.dae"/>
       </geometry>
     </visual>

Commit message: Add geotagged tif of the inspection world, move the origin to be vaguely representative of a lake in northern Alberta

File: cpr_inspection_gazebo/urdf/inspection_geometry.urdf.xacro (robot description, xacro)
@@ -8,5 +8,5 @@
     </inertial>
     <visual>
-      <origin xyz="0 0 0" rpy="0 0 0"/>
+      <origin xyz="0 0 0" rpy="0 0 1.5707963267948966"/>
       <geometry>
         <mesh filename="package://cpr_inspection_gazebo/meshes/inspection_world.dae"/>
@@ -14,5 +14,5 @@
     </visual>
     <visual>
-      <origin xyz="0 0 0" rpy="0 0 0"/>
+      <origin xyz="0 0 0" rpy="0 0 1.5707963267948966"/>
       <geometry>
         <mesh filename="package://cpr_inspection_gazebo/meshes/inspection_water.dae"/>
@@ -20,5 +20,5 @@
     </visual>
     <collision>
-      <origin xyz="0 0 0" rpy="0 0 0"/>
+      <origin xyz="0 0 0" rpy="0 0 1.5707963267948966"/>
       <geometry>
         <mesh filename="package://cpr_inspection_gazebo/meshes/inspection_world.dae"/>

Commit message: Increase the horizontal scale of the world to make the hill proportionally shallower. Re-tag the geotif with updated coordiantes

File: cpr_inspection_gazebo/urdf/inspection_geometry.urdf.xacro (robot description, xacro)
@@ -10,5 +10,5 @@
       <origin xyz="0 0 0" rpy="0 0 1.5707963267948966"/>
       <geometry>
-        <mesh filename="package://cpr_inspection_gazebo/meshes/inspection_world.dae"/>
+        <mesh filename="package://cpr_inspection_gazebo/meshes/inspection_world.dae" scale="2 2 1"/>
       </geometry>
     </visual>
@@ -16,5 +16,5 @@
       <origin xyz="0 0 0" rpy="0 0 1.5707963267948966"/>
       <geometry>
-        <mesh filename="package://cpr_inspection_gazebo/meshes/inspection_water.dae"/>
+        <mesh filename="package://cpr_inspection_gazebo/meshes/inspection_water.dae" scale="2 2 1"/>
       </geometry>
     </visual>
@@ -22,5 +22,5 @@
       <origin xyz="0 0 0" rpy="0 0 1.5707963267948966"/>
       <geometry>
-        <mesh filename="package://cpr_inspection_gazebo/meshes/inspection_world.dae"/>
+        <mesh filename="package://cpr_inspection_gazebo/meshes/inspection_world.dae" scale="2 2 1"/>
       </geometry>
       <surface>

Commit message: Add the base station object on the shore of the lake

File: cpr_inspection_gazebo/urdf/inspection_geometry.urdf.xacro (robot description, xacro)
@@ -34,4 +34,8 @@
     </collision>
   </link>
+  <xacro:include filename="$(find cpr_accessories_gazebo)/urdf/base_station.urdf.xacro" />
+  <xacro:cpr_base_station name="base_station" parent="inspection_world_link">
+    <origin xyz="-12 0 1" rpy="0 0 0" />
+  </xacro:cpr_base_station>
   <gazebo> <static>true</static></gazebo>
 </robot>

Commit message: Adjust the orchard and inspection worlds to use ENU coordinates for the world frame. Fix the robot spawn points, GPS base-station locations, and default camera orientations accordingly

File: cpr_inspection_gazebo/urdf/inspection_geometry.urdf.xacro (robot description, xacro)
@@ -8,5 +8,5 @@
     </inertial>
     <visual>
-      <origin xyz="0 0 0" rpy="0 0 1.5707963267948966"/>
+      <origin xyz="0 0 0" rpy="0 0 3.141592653589793"/>
       <geometry>
         <mesh filename="package://cpr_inspection_gazebo/meshes/inspection_world.dae" scale="2 2 1"/>
@@ -14,5 +14,5 @@
     </visual>
     <visual>
-      <origin xyz="0 0 0" rpy="0 0 1.5707963267948966"/>
+      <origin xyz="0 0 0" rpy="0 0 3.141592653589793"/>
       <geometry>
         <mesh filename="package://cpr_inspection_gazebo/meshes/inspection_water.dae" scale="2 2 1"/>
@@ -20,5 +20,5 @@
     </visual>
     <collision>
-      <origin xyz="0 0 0" rpy="0 0 1.5707963267948966"/>
+      <origin xyz="0 0 0" rpy="0 0 3.141592653589793"/>
       <geometry>
         <mesh filename="package://cpr_inspection_gazebo/meshes/inspection_world.dae" scale="2 2 1"/>
@@ -36,5 +36,5 @@
   <xacro:include filename="$(find cpr_accessories_gazebo)/urdf/base_station.urdf.xacro" />
   <xacro:cpr_base_station name="base_station" parent="inspection_world_link">
-    <origin xyz="-12 0 1" rpy="0 0 0" />
+    <origin xyz="0 -12 1" rpy="0 0 0" />
   </xacro:cpr_base_station>
   <gazebo> <static>true</static></gazebo>

File: cpr_orchard_gazebo/urdf/orchard_geometry.urdf.xacro (robot description, xacro)
@@ -8,5 +8,5 @@
     </inertial>
     <visual>
-      <origin xyz="0 0 0" rpy="0 0 0"/>
+      <origin xyz="0 0 0" rpy="0 0 1.5707963267948966"/>
       <geometry>
         <mesh filename="package://cpr_orchard_gazebo/meshes/orchard_world.dae"/>
@@ -14,5 +14,5 @@
     </visual>
     <visual>
-      <origin xyz="0 0 0" rpy="0 0 0"/>
+      <origin xyz="0 0 0" rpy="0 0 1.5707963267948966"/>
       <geometry>
         <mesh filename="package://cpr_orchard_gazebo/meshes/orchard_trunks.dae"/>
@@ -20,5 +20,5 @@
     </visual>
     <visual>
-      <origin xyz="0 0 0" rpy="0 0 0"/>
+      <origin xyz="0 0 0" rpy="0 0 1.5707963267948966"/>
       <geometry>
         <mesh filename="package://cpr_orchard_gazebo/meshes/orchard_leaves.dae"/>
@@ -26,5 +26,5 @@
     </visual>
     <collision>
-      <origin xyz="0 0 0" rpy="0 0 0"/>
+      <origin xyz="0 0 0" rpy="0 0 1.5707963267948966"/>
       <geometry>
         <mesh filename="package://cpr_orchard_gazebo/meshes/orchard_world.dae"/>
@@ -40,5 +40,5 @@
     </collision>
     <collision>
-      <origin xyz="0 0 0" rpy="0 0 0"/>
+      <origin xyz="0 0 0" rpy="0 0 1.5707963267948966"/>
       <geometry>
         <mesh filename="package://cpr_orchard_gazebo/meshes/orchard_trunks.dae"/>
@@ -49,5 +49,5 @@
   <xacro:include filename="$(find cpr_accessories_gazebo)/urdf/base_station.urdf.xacro" />
   <xacro:cpr_base_station name="base_station" parent="orchard_world_link">
-    <origin xyz="1 2 0" />
+    <origin xyz="-2 1 0" />
   </xacro:cpr_base_station>
 </robot>
