Commit message: Add a new accessories package with the charge dock and base station. Add view_world.launch files to all relevant packages so you can view the environment without spinning up Gazebo. Add the wireless charge dock and base station to the agriculture world

File: cpr_agriculture_gazebo/urdf/agriculture_geometry.urdf.xacro (robot description, xacro)
@@ -28,4 +28,12 @@
     </collision>
   </link>
+  <xacro:include filename="$(find cpr_accessories_gazebo)/urdf/base_station.urdf.xacro" />
+  <xacro:cpr_base_station name="base_station" parent="agriculture_world_link">
+    <origin xyz="40 17 0.7" />
+  </xacro:cpr_base_station>
+  <xacro:include  filename="$(find cpr_accessories_gazebo)/urdf/charge_dock.urdf.xacro" />
+  <xacro:cpr_charge_dock name="charge_dock" parent="agriculture_world_link">
+    <origin xyz="-8 4 -0.2" rpy="0 0 -1.5707963267948966" />
+  </xacro:cpr_charge_dock>
   <gazebo> <static>true</static></gazebo>
 </robot>

File: cpr_obstacle_gazebo/urdf/obstacle_geometry.urdf.xacro (robot description, xacro)
@@ -1,4 +1,4 @@
 <?xml version="1.0" ?>
-<robot xmlns:xacro="http://wiki.ros.org/xacro">
+<robot xmlns:xacro="http://wiki.ros.org/xacro" name="obstacle_world">
   <xacro:arg name="world_scale" default="1.0" />
   <xacro:arg name="walls" default="true" />

Commit message: Rotate the world so it aligns with ENU

File: cpr_agriculture_gazebo/urdf/agriculture_geometry.urdf.xacro (robot description, xacro)
@@ -8,5 +8,5 @@
     </inertial>
     <visual>
-      <origin xyz="0 0 0" rpy="0 0 0"/>
+      <origin xyz="0 0 0" rpy="0 0 3.141592653589793"/>
       <geometry>
         <mesh filename="package://cpr_agriculture_gazebo/meshes/agriculture_world.dae"/>
@@ -14,5 +14,5 @@
     </visual>
     <collision>
-      <origin xyz="0 0 0" rpy="0 0 0"/>
+      <origin xyz="0 0 0" rpy="0 0 3.141592653589793"/>
       <geometry>
         <mesh filename="package://cpr_agriculture_gazebo/meshes/agriculture_world.dae"/>
@@ -30,9 +30,9 @@
   <xacro:include filename="$(find cpr_accessories_gazebo)/urdf/base_station.urdf.xacro" />
   <xacro:cpr_base_station name="base_station" parent="agriculture_world_link">
-    <origin xyz="40 17 0.7" />
+    <origin xyz="-40 -17 0.7" />
   </xacro:cpr_base_station>
   <xacro:include  filename="$(find cpr_accessories_gazebo)/urdf/charge_dock.urdf.xacro" />
   <xacro:cpr_charge_dock name="charge_dock" parent="agriculture_world_link">
-    <origin xyz="-8 4 -0.2" rpy="0 0 -1.5707963267948966" />
+    <origin xyz="8 -4 0.2" rpy="0 0 1.5707963267948966" />
   </xacro:cpr_charge_dock>
   <gazebo> <static>true</static></gazebo>

Commit message: Rotate the world so that north is along the X axis

File: cpr_agriculture_gazebo/urdf/agriculture_geometry.urdf.xacro (robot description, xacro)
@@ -7,6 +7,9 @@
       <inertia ixx="1" ixy="0" ixz="0" iyy="1" iyz="0" izz="1"/>
     </inertial>
+    <!--
+      Align the world geometry so that X+ is north and Y+ is west
+    -->
     <visual>
-      <origin xyz="0 0 0" rpy="0 0 3.141592653589793"/>
+      <origin xyz="0 0 0" rpy="0 0 1.5707963267948966"/>
       <geometry>
         <mesh filename="package://cpr_agriculture_gazebo/meshes/agriculture_world.dae"/>
@@ -14,5 +17,5 @@
     </visual>
     <collision>
-      <origin xyz="0 0 0" rpy="0 0 3.141592653589793"/>
+      <origin xyz="0 0 0" rpy="0 0 1.5707963267948966"/>
       <geometry>
         <mesh filename="package://cpr_agriculture_gazebo/meshes/agriculture_world.dae"/>
@@ -30,9 +33,9 @@
   <xacro:include filename="$(find cpr_accessories_gazebo)/urdf/base_station.urdf.xacro" />
   <xacro:cpr_base_station name="base_station" parent="agriculture_world_link">
-    <origin xyz="-40 -17 0.7" />
+    <origin xyz="-17 40 0.7" />
   </xacro:cpr_base_station>
   <xacro:include  filename="$(find cpr_accessories_gazebo)/urdf/charge_dock.urdf.xacro" />
   <xacro:cpr_charge_dock name="charge_dock" parent="agriculture_world_link">
-    <origin xyz="8 -4 0.2" rpy="0 0 1.5707963267948966" />
+    <origin xyz="-4 -8 -0.2" rpy="0 0 0" />
   </xacro:cpr_charge_dock>
   <gazebo> <static>true</static></gazebo>

Commit message: Fix the world geometry to use ENU, fix the sun direction so it makes sense for the world

File: cpr_agriculture_gazebo/urdf/agriculture_geometry.urdf.xacro (robot description, xacro)
@@ -8,8 +8,8 @@
     </inertial>
     <!--
-      Align the world geometry so that X+ is north and Y+ is west
+      Align the world geometry so that X+ is east and Y+ is north (ENU)
     -->
     <visual>
-      <origin xyz="0 0 0" rpy="0 0 1.5707963267948966"/>
+      <origin xyz="0 0 0" rpy="0 0 ${pi}"/>
       <geometry>
         <mesh filename="package://cpr_agriculture_gazebo/meshes/agriculture_world.dae"/>
@@ -17,5 +17,5 @@
     </visual>
     <collision>
-      <origin xyz="0 0 0" rpy="0 0 1.5707963267948966"/>
+      <origin xyz="0 0 0" rpy="0 0 ${pi}"/>
       <geometry>
         <mesh filename="package://cpr_agriculture_gazebo/meshes/agriculture_world.dae"/>

Commit message: Move the wireless charge dock back outside

File: cpr_agriculture_gazebo/urdf/agriculture_geometry.urdf.xacro (robot description, xacro)
@@ -37,5 +37,5 @@
   <xacro:include  filename="$(find cpr_accessories_gazebo)/urdf/charge_dock.urdf.xacro" />
   <xacro:cpr_charge_dock name="charge_dock" parent="agriculture_world_link">
-    <origin xyz="-4 -8 -0.2" rpy="0 0 0" />
+    <origin xyz="8 -4 -0.2" rpy="0 0 1.5707963267948966" />
   </xacro:cpr_charge_dock>
   <gazebo> <static>true</static></gazebo>

Commit message: Fix the location of the base station in the agriculture world

File: cpr_agriculture_gazebo/urdf/agriculture_geometry.urdf.xacro (robot description, xacro)
@@ -33,5 +33,5 @@
   <xacro:include filename="$(find cpr_accessories_gazebo)/urdf/base_station.urdf.xacro" />
   <xacro:cpr_base_station name="base_station" parent="agriculture_world_link">
-    <origin xyz="-17 40 0.7" />
+    <origin xyz="-40 -17 0.7" />
   </xacro:cpr_base_station>
   <xacro:include  filename="$(find cpr_accessories_gazebo)/urdf/charge_dock.urdf.xacro" />
