Commit message: enable dock in empty world

File: cpr_empty_gazebo/urdf/empty_geometry.urdf.xacro (robot description, xacro)
@@ -35,10 +35,11 @@
     <origin xyz="50 50 0" />
   </xacro:cpr_base_station>
-  <!-- Temporarily disabled; will be re-enabled later
+  <xacro:arg name="dock_x"   default="$(optenv CPR_SIMULATION_DOCK_X 10.0)"/>
+  <xacro:arg name="dock_y"   default="$(optenv CPR_SIMULATION_DOCK_Y 10.0)"/>
+  <xacro:arg name="dock_yaw" default="$(optenv CPR_SIMULATION_DOCK_YAW 0.0)"/>
   <xacro:include  filename="$(find cpr_accessories_gazebo)/urdf/charge_dock.urdf.xacro" />
   <xacro:cpr_charge_dock name="charge_dock" parent="empty_world_link">
-    <origin xyz="10 -10 0" rpy="0 0 2.356194490192345"/>
+    <origin xyz="$(arg dock_x) $(arg dock_y) 0" rpy="0 0 $(arg dock_yaw)"/>
   </xacro:cpr_charge_dock>
-  -->
   <gazebo> <static>true</static></gazebo>
 </robot>
